Commit message: Little changes xD

File: test/models/r6bot/r6bot.urdf (robot description, URDF)
Before this commit: robot r6bot, 10 links, 9 joints
Links:
- link base_link: geometry collision mesh filename=package://multi_end_effector_kinematics/models/r6bot/meshes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; visual mesh filename=package://multi_end_effector_kinematics/models/r6bot/meshes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
- link link_1: geometry collision mesh filename=package://multi_end_effector_kinematics/models/r6bot/meshes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; visual mesh filename=package://multi_end_effector_kinematics/models/r6bot/meshes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
- link link_2: geometry collision mesh filename=package://multi_end_effector_kinematics/models/r6bot/meshes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; visual mesh filename=package://multi_end_effector_kinematics/models/r6bot/meshes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
- link link_3: geometry collision mesh filename=package://multi_end_effector_kinematics/models/r6bot/meshes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; visual mesh filename=package://multi_end_effector_kinematics/models/r6bot/meshes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
- link link_4: geometry collision mesh filename=package://multi_end_effector_kinematics/models/r6bot/meshes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; visual mesh filename=package://multi_end_effector_kinematics/models/r6bot/meshes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
- link link_5: geometry collision mesh filename=package://multi_end_effector_kinematics/models/r6bot/meshes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; visual mesh filename=package://multi_end_effector_kinematics/models/r6bot/meshes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
- link link_6: geometry collision mesh filename=package://multi_end_effector_kinematics/models/r6bot/meshes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; visual mesh filename=package://multi_end_effector_kinematics/models/r6bot/meshes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

File: test/models/r6bot/r6bot.urdf.xacro (robot description, xacro)
@@ -2,5 +2,5 @@
 <robot xmlns:xacro="http://wiki.ros.org/xacro" name="r6bot">
   <!-- Import r6bot macro -->
-  <xacro:include filename="$(find lrt_inverse_kinematics)/models/r6bot/urdf/r6bot_description.urdf.xacro"/>
+  <xacro:include filename="$(find multi_end_effector_kinematics)/models/r6bot/urdf/r6bot_description.urdf.xacro"/>
   <!-- create link fixed to the "world" -->
   <link name="world"/>

File: test/models/r6bot/urdf/r6bot_description.urdf.xacro (robot description, xacro)
@@ -3,10 +3,10 @@
   <xacro:macro name="r6bot_description">
   <!-- helper macro -->
-  <xacro:include filename="$(find lrt_inverse_kinematics)/models/r6bot/urdf/inc/create_link.xacro"/>
+  <xacro:include filename="$(find multi_end_effector_kinematics)/models/r6bot/urdf/inc/create_link.xacro"/>
   <xacro:create_link
       link_name="base_link"
       xyz_offset="0 0 0"
       rpy_offset="0 0 0"
-      mesh_package="lrt_inverse_kinematics/models/r6bot"
+      mesh_package="multi_end_effector_kinematics/models/r6bot"
       mesh_name="link_0"
   />
@@ -15,5 +15,5 @@
       xyz_offset="0 0 0"
       rpy_offset="0 0 0"
-      mesh_package="lrt_inverse_kinematics/models/r6bot"
+      mesh_package="multi_end_effector_kinematics/models/r6bot"
       mesh_name="link_1"
   />
@@ -22,5 +22,5 @@
       xyz_offset="0 0 0"
       rpy_offset="0 0 0"
-      mesh_package="lrt_inverse_kinematics/models/r6bot"
+      mesh_package="multi_end_effector_kinematics/models/r6bot"
       mesh_name="link_2"
   />
@@ -29,5 +29,5 @@
       xyz_offset="0 0 0"
       rpy_offset="0 0 0"
-      mesh_package="lrt_inverse_kinematics/models/r6bot"
+      mesh_package="multi_end_effector_kinematics/models/r6bot"
       mesh_name="link_3"
   />
@@ -36,5 +36,5 @@
       xyz_offset="0 0 0"
       rpy_offset="0 0 0"
-      mesh_package="lrt_inverse_kinematics/models/r6bot"
+      mesh_package="multi_end_effector_kinematics/models/r6bot"
       mesh_name="link_4"
   />
@@ -43,5 +43,5 @@
       xyz_offset="0 0 0"
       rpy_offset="0 0 0"
-      mesh_package="lrt_inverse_kinematics/models/r6bot"
+      mesh_package="multi_end_effector_kinematics/models/r6bot"
       mesh_name="link_5"
   />
@@ -50,5 +50,5 @@
       xyz_offset="0 0 0"
       rpy_offset="0 0 0"
-      mesh_package="lrt_inverse_kinematics/models/r6bot"
+      mesh_package="multi_end_effector_kinematics/models/r6bot"
       mesh_name="link_6"
   />
